Commit message: updated slx,stl,urdf

File: Team7_Milestone2/Script Folder/final_robot.urdf (robot description, URDF)
Before this commit: robot rr, 5 links, 4 joints
Links:
- link Gripper: geometry collision mesh filename=package://mokhito/meshes/Gripper.STL; visual mesh filename=package://mokhito/meshes/Gripper.STL
- link Link1: geometry collision mesh filename=package://mokhito/meshes/Link1.STL; visual mesh filename=package://mokhito/meshes/Link1.STL
- link Link2: geometry collision mesh filename=package://mokhito/meshes/Link2.STL; visual mesh filename=package://mokhito/meshes/Link2.STL
- link Link3: geometry collision mesh filename=package://mokhito/meshes/Link3.STL; visual mesh filename=package://mokhito/meshes/Link3.STL
- link base_link: geometry collision mesh filename=package://mokhito/meshes/base_link.STL; visual mesh filename=package://mokhito/meshes/base_link.STL
Joints:
- joint Joint1: origin xyz=-0.0520277439177293 -0.0678255172812337 0.0781521980886112 rpy=0 0 0 -> xyz=-0.0520277439177293 -0.0678255172812337 0.0781521980886112 rpy=0 0 1.5707963267949
- joint Joint2: origin xyz=0 0 0.0435500000000015 rpy=1.5707963267949 0 1.5707963267949 -> xyz=0 0 0.0435500000000015 rpy=1.5707963267949 0 0
- joint Joint3: origin xyz=0.00764208484451164 0.139791267750278 0 rpy=0 0 -1.55524821349945 -> xyz=0.00764208484451164 0.139791267750278 0 rpy=0 0 1.58634444009034
- joint Joint4: origin xyz=-0.134100000000004 -0.000353979969758569 0 rpy=-0.0245233381074276 -0.00151760690316946 3.07979966379466 -> xyz=0.134100000000004 0.000353979969758569 0 rpy=-0.0245233381074276 -0.00151760690316946 -0.061792989795138
